Commit message: it moves

File: config/gummi.urdf (robot description, URDF)
Before this commit: robot gummi, 43 links, 42 joints
Links:
- removed link base
- added link right_base_link, mass 0.335467320988356; collision mesh filename=package://gummi_rightbase_template/meshes/base_link.STL; visual mesh filename=package://gummi_rightbase_template/meshes/base_link.STL
- link base_link: mass 0.335467320988356 -> None; geometry 
Joints:
- joint leftbase_displacement: origin xyz=-0.2 0 0 rpy=0 0 0 -> xyz=-0.2 0 0 rpy=-3.14 0 0; parent base -> base_link
- joint rightbase_displacement: child base_link -> right_base_link; parent base -> base_link
- joint shoulder_yaw: parent base_link -> right_base_link

File: xacro/gummi_rig.urdf.xacro (robot description, xacro)
@@ -2,18 +2,18 @@
 <robot
   name="gummi" xmlns:xacro="http://www.ros.org/wiki/xacro">
-  <link name="base"/>
-<xacro:include filename="$(env GUMMI_LEFTBASEPATH)/xacro/gummi_description.urdf.xacro" />
-<xacro:include filename="$(env GUMMI_RIGHTBASEPATH)/xacro/gummi_description.urdf.xacro" />
+<xacro:include filename="$(env GUMMI_LEFTBASEPATH)/xacro/gummi_left.urdf.xacro" />
+<xacro:include filename="$(env GUMMI_RIGHTBASEPATH)/xacro/gummi_right.urdf.xacro" />
+<link name="base_link"/>
+<joint name="rightbase_displacement" type="fixed">
+  <origin rpy="0 0 0" xyz="0.2 0 0"/>
+  <parent link="base_link"/>
+  <child link="right_base_link"/>
+  <axis xyz="0 0 0"/>
+</joint>
 <joint name="leftbase_displacement" type="fixed">
-  <origin rpy="0 0 0" xyz="-0.2 0 0"/>
-  <parent link="base"/>
+  <origin rpy="-3.14 0 0" xyz="-0.2 0 0"/>
+  <parent link="base_link"/>
   <child link="left_base_link"/>
   <axis xyz="0 0 0"/>
 </joint>
-<joint name="rightbase_displacement" type="fixed">
-  <origin rpy="0 0 0" xyz="0.2 0 0"/>
-  <parent link="base"/>
-  <child link="base_link"/>
-  <axis xyz="0 0 0"/>
-</joint>
 </robot>

Commit message: preparing for namespacing /left

File: config/gummi.urdf (robot description, URDF)
Before this commit: robot gummi, 43 links, 42 joints
Links:
- removed link dummyleft_gripper
- removed link left_base_link
- removed link left_i1
- removed link left_i2
- removed link left_i3
- removed link left_i4
- removed link left_i5
- removed link left_lowerarm
- removed link left_lowerarm_preroll_d
- removed link left_lowerarm_preroll_u
- removed link left_shoulder
- removed link left_shoulder_pitch_back_pulley
- removed link left_shoulder_pitch_front_pulley
- removed link left_shoulder_preroll
- removed link left_shoulder_roll_bottom_pulley
- removed link left_shoulder_roll_top_pulley
- removed link left_upperarm
- removed link left_upperarm_biceps_pulley
- removed link left_upperarm_preroll
- removed link left_upperarm_triceps_pulley
- removed link left_wrist
- added link left/base_link, mass 0.335467320988356; collision mesh filename=package://gummi_leftbase_template/meshes/base_link.STL; visual mesh filename=package://gummi_leftbase_template/meshes/base_link.STL
- added link left/fake_gripper
- added link left/lowerarm, mass 0.258562959800175; collision mesh filename=package://gummi_leftee_popeye_wirecutter/meshes/lowerarm.STL; visual mesh filename=package://gummi_leftee_popeye_wirecutter/meshes/lowerarm.STL
- added link left/lowerarm_preroll_d, mass 0.106215245171982; collision mesh filename=package://gummi_leftee_popeye_wirecutter/meshes/lowerarm_pr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; visual mesh filename=package://gummi_leftee_popeye_wirecutter/meshes/lowerarm_pr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
- added link left/lowerarm_preroll_u, mass 0.034447; collision mesh filename=package://gummi_leftbase_template/meshes/lowerarm_preroll_u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; visual mesh filename=package://gummi_leftbase_template/meshes/lowerarm_preroll_u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
- added link left/shoulder, mass 0.32611; collision mesh filename=package://gummi_leftbase_template/meshes/shoulder.STL; visual mesh filename=package://gummi_leftbase_template/meshes/shoulder.STL
- added link left/shoulder_pitch_back_pulley, mass 0.027251; collision mesh filename=package://gummi_leftbase_template/meshes/shoulder_pitch_bac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; visual mesh filename=package://gummi_leftbase_template/meshes/shoulder_pitch_bac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
- added link left/shoulder_pitch_front_pulley, mass 0.027251; collision mesh filename=package://gummi_leftbase_template/meshes/shoulder_pitch_fro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; visual mesh filename=package://gummi_leftbase_template/meshes/shoulder_pitch_fro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
- added link left/shoulder_preroll, mass 0.77225; collision mesh filename=package://gummi_leftbase_template/meshes/shoulder_preroll.S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; visual mesh filename=package://gummi_leftbase_template/meshes/shoulder_preroll.S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
- added link left/shoulder_roll_bottom_pulley, mass 0.01522; collision mesh filename=package://gummi_leftbase_template/meshes/shoulder_roll_bott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; visual mesh filename=package://gummi_leftbase_template/meshes/shoulder_roll_bott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
- added link left/shoulder_roll_top_pulley, mass 0.01522; collision mesh filename=package://gummi_leftbase_template/meshes/shoulder_roll_top_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; visual mesh filename=package://gummi_leftbase_template/meshes/shoulder_roll_top_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
- added link left/tool
- added link left/upperarm, mass 0.26501; collision mesh filename=package://gummi_leftbase_template/meshes/upperarm.STL; visual mesh filename=package://gummi_leftbase_template/meshes/upperarm.STL
- added link left/upperarm_biceps_pulley, mass 0.01522; collision mesh filename=package://gummi_leftbase_template/meshes/upperarm_biceps_pu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; visual mesh filename=package://gummi_leftbase_template/meshes/upperarm_biceps_pu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
- added link left/upperarm_preroll, mass 0.11889; collision mesh filename=package://gummi_leftbase_template/meshes/upperarm_preroll.S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; visual mesh filename=package://gummi_leftbase_template/meshes/upperarm_preroll.S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
- added link left/upperarm_triceps_pulley, mass 0.01522; collision mesh filename=package://gummi_leftbase_template/meshes/upperarm_triceps_p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; visual mesh filename=package://gummi_leftbase_template/meshes/upperarm_triceps_p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
- added link left/wrist, mass 1.33735316789728; collision mesh filename=package://gummi_leftee_popeye_wirecutter/meshes/wrist.STL; visual mesh filename=package://gummi_leftee_popeye_wirecutter/meshes/wrist.STL
- added link left/wrist_ext_pulley, mass 0.0159623836902443; collision mesh filename=package://gummi_leftee_popeye_wirecutter/meshes/wrist_ext_p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; visual mesh filename=package://gummi_leftee_popeye_wirecutter/meshes/wrist_ext_p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
- added link left/wrist_flex_pulley, mass 0.0159623838254221; collision mesh filename=package://gummi_leftee_popeye_wirecutter/meshes/wrist_flex_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; visual mesh filename=package://gummi_leftee_popeye_wirecutter/meshes/wrist_flex_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
Joints:
- removed joint left_elbow
- removed joint left_fastswitch
- removed joint left_forearm_roll
- removed joint left_gripper
- removed joint left_i1f
- removed joint left_i2f
- removed joint left_i3f
- removed joint left_i4f
- removed joint left_i5f
- removed joint left_shoulder_pitch
- removed joint left_shoulder_pitch_back_pulley_joint
- removed joint left_shoulder_pitch_pulley_front_joint
- removed joint left_shoulder_roll
- removed joint left_shoulder_roll_bottom_pulley
- removed joint left_shoulder_roll_top_pulley_joint
- removed joint left_shoulder_yaw
- removed joint left_upperarm_biceps_pulley_joint
- removed joint left_upperarm_roll
- removed joint left_upperarm_triceps_pulley_joint
- removed joint left_wrist_pitch
- added joint left/coupling_tool: type fixed, parent left/wrist, child left/tool, origin xyz=0.25 0 0.25 rpy=0 0 0, axis 1 0 0, limit lower=0 upper=1 effort=0 velocity=0
- added joint left/elbow: type revolute, parent left/upperarm, child left/lowerarm_preroll_u, origin xyz=-0.006 0.0184 -0.23533 rpy=0 0 0, axis 0 -1 0, limit lower=-0.75 upper=0.35 effort=0 velocity=0
- added joint left/fastswitch: type fixed, parent left/lowerarm_preroll_u, child left/lowerarm_preroll_d, origin xyz=0.057 -0.019 -0.005 rpy=0 0 0, axis 0 0 0
- added joint left/forearm_roll: type revolute, parent left/lowerarm_preroll_d, child left/lowerarm, origin xyz=0.0073428 -0.00024663 -0.037992 rpy=0 0 0, axis 1 0 0, limit lower=-1 upper=1 effort=0 velocity=0
- added joint left/gripper: type prismatic, parent left/wrist, child left/fake_gripper, origin xyz=0 0 0 rpy=0 0 0, axis 0 0 1, limit lower=0 upper=1 effort=0 velocity=0
- added joint left/shoulder_pitch: type revolute, parent left/shoulder, child left/upperarm_preroll, origin xyz=-0.024 -0.17679 8.6827E-05 rpy=0 0 0, axis -1 0 0, limit lower=-0.15 upper=1.1 effort=0 velocity=0
- added joint left/shoulder_pitch_back_pulley_joint: type fixed, parent left/shoulder_preroll, child left/shoulder_pitch_back_pulley, origin xyz=-0.067526 -0.024095 0.044 rpy=0 0 0, axis 0 0 0
- added joint left/shoulder_pitch_pulley_front_joint: type fixed, parent left/shoulder_preroll, child left/shoulder_pitch_front_pulley, origin xyz=0.067474 -0.024095 0.044 rpy=0 0 0, axis 0 0 0
- added joint left/shoulder_roll: type revolute, parent left/shoulder_preroll, child left/shoulder, origin xyz=-2.6378E-05 0.057605 0.1302 rpy=0 0 0, axis 0 -1 0, limit lower=-0.95 upper=2.3 effort=0 velocity=0
- added joint left/shoulder_roll_bottom_pulley: type fixed, parent left/shoulder, child left/shoulder_roll_bottom_pulley, origin xyz=-0.0208 -0.06848 -0.043 rpy=0 0 0, axis 0 0 -1, limit effort=0 velocity=0
- added joint left/shoulder_roll_top_pulley_joint: type fixed, parent left/shoulder, child left/shoulder_roll_top_pulley, origin xyz=0.0208 -0.06848 0.043 rpy=0 0 0, axis 0 0 0
- added joint left/shoulder_yaw: type revolute, parent left/base_link, child left/shoulder_preroll, origin xyz=-0.00027025 -0.10997 0.008 rpy=0 0 0, axis 0 0 1, limit lower=-0.75 upper=1 effort=0 velocity=0
- added joint left/upperarm_biceps_pulley_joint: type fixed, parent left/upperarm, child left/upperarm_biceps_pulley, origin xyz=0.0375 0 -0.10243 rpy=0 0 0, axis 0 0 0
- added joint left/upperarm_roll: type revolute, parent left/upperarm_preroll, child left/upperarm, origin xyz=0.056992 -0.010088 -0.035587 rpy=0 0 0, axis 0 0 -1, limit lower=-1.56 upper=1.56 effort=0 velocity=0
- added joint left/upperarm_triceps_pulley_joint: type fixed, parent left/upperarm, child left/upperarm_triceps_pulley, origin xyz=-0.0435 0 -0.12843 rpy=0 0 0, axis -1 0 0, limit effort=0 velocity=0
- added joint left/wrist_ext_pulley_joint: type continuous, parent left/lowerarm, child left/wrist_ext_pulley, origin xyz=0.1061 0.04025 -0.02035 rpy=0 0 0, axis 0 -1 0, mimic joint=left/wrist_pitch
- added joint left/wrist_flex_pulley_joint: type continuous, parent left/lowerarm, child left/wrist_flex_pulley, origin xyz=0.1061 -0.04025 0.02035 rpy=0 0 0, axis 0 -1 0, mimic joint=left/wrist_pitch
- added joint left/wrist_pitch: type revolute, parent left/lowerarm, child left/wrist, origin xyz=0.18238 -0.028 0 rpy=0 0 0, axis 0 1 0, limit lower=-1 upper=1 effort=0 velocity=0
- joint leftbase_displacement: child left_base_link -> left/base_link

File: xacro/gummi_rig.urdf.xacro (robot description, xacro)
@@ -14,5 +14,5 @@
   <origin rpy="-3.14 0 0" xyz="-0.2 0 0"/>
   <parent link="base_link"/>
-  <child link="left_base_link"/>
+  <child link="left/base_link"/>
   <axis xyz="0 0 0"/>
 </joint>

Commit message: rig with both arms in namespaces

File: config/gummi.urdf (robot description, URDF)
Before this commit: robot gummi, 41 links, 40 joints
Links:
- removed link dummygripper
- removed link i1
- removed link i2
- removed link i3
- removed link i4
- removed link i5
- removed link lowerarm
- removed link lowerarm_preroll_d
- removed link lowerarm_preroll_u
- removed link right_base_link
- removed link shoulder
- removed link shoulder_pitch_back_pulley
- removed link shoulder_pitch_front_pulley
- removed link shoulder_preroll
- removed link shoulder_roll_bottom_pulley
- removed link shoulder_roll_top_pulley
- removed link upperarm
- removed link upperarm_biceps_pulley
- removed link upperarm_preroll
- removed link upperarm_triceps_pulley
- removed link wrist
- added link right/base_link, mass 0.335467320988356; collision mesh filename=package://gummi_rightbase_template/meshes/base_link.STL; visual mesh filename=package://gummi_rightbase_template/meshes/base_link.STL
- added link right/dummygripper
- added link right/i1, mass 0.00632408233084942; collision mesh filename=package://gummi_rightee_handshake/meshes/i1.STL; visual mesh filename=package://gummi_rightee_handshake/meshes/i1.STL
- added link right/i2, mass 0.00478605585780196; collision mesh filename=package://gummi_rightee_handshake/meshes/i2.STL; visual mesh filename=package://gummi_rightee_handshake/meshes/i2.STL
- added link right/i3, mass 0.00575461720344836; collision mesh filename=package://gummi_rightee_handshake/meshes/i3.STL; visual mesh filename=package://gummi_rightee_handshake/meshes/i3.STL
- added link right/i4, mass 0.00478456052942582; collision mesh filename=package://gummi_rightee_handshake/meshes/i4.STL; visual mesh filename=package://gummi_rightee_handshake/meshes/i4.STL
- added link right/i5, mass 0.00396686667442233; collision mesh filename=package://gummi_rightee_handshake/meshes/i5.STL; visual mesh filename=package://gummi_rightee_handshake/meshes/i5.STL
- added link right/lowerarm, mass 0.214658222402075; collision mesh filename=package://gummi_rightee_handshake/meshes/lowerarm.STL; visual mesh filename=package://gummi_rightee_handshake/meshes/lowerarm.STL
- added link right/lowerarm_preroll_d, mass 0.0573922743530686; collision mesh filename=package://gummi_rightee_handshake/meshes/lowerarm_preroll_d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; visual mesh filename=package://gummi_rightee_handshake/meshes/lowerarm_preroll_d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
- added link right/lowerarm_preroll_u, mass 0.034447; collision mesh filename=package://gummi_rightbase_template/meshes/lowerarm_preroll_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; visual mesh filename=package://gummi_rightbase_template/meshes/lowerarm_preroll_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
- added link right/shoulder, mass 0.32611; collision mesh filename=package://gummi_rightbase_template/meshes/shoulder.STL; visual mesh filename=package://gummi_rightbase_template/meshes/shoulder.STL
- added link right/shoulder_pitch_back_pulley, mass 0.027251; collision mesh filename=package://gummi_rightbase_template/meshes/shoulder_pitch_ba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; visual mesh filename=package://gummi_rightbase_template/meshes/shoulder_pitch_ba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
- added link right/shoulder_pitch_front_pulley, mass 0.027251; collision mesh filename=package://gummi_rightbase_template/meshes/shoulder_pitch_fr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; visual mesh filename=package://gummi_rightbase_template/meshes/shoulder_pitch_fr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
- added link right/shoulder_preroll, mass 0.77225; collision mesh filename=package://gummi_rightbase_template/meshes/shoulder_preroll.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; visual mesh filename=package://gummi_rightbase_template/meshes/shoulder_preroll.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
- added link right/shoulder_roll_bottom_pulley, mass 0.01522; collision mesh filename=package://gummi_rightbase_template/meshes/shoulder_roll_bot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; visual mesh filename=package://gummi_rightbase_template/meshes/shoulder_roll_bot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
- added link right/shoulder_roll_top_pulley, mass 0.01522; collision mesh filename=package://gummi_rightbase_template/meshes/shoulder_roll_top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; visual mesh filename=package://gummi_rightbase_template/meshes/shoulder_roll_top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
- added link right/upperarm, mass 0.26501; collision mesh filename=package://gummi_rightbase_template/meshes/upperarm.STL; visual mesh filename=package://gummi_rightbase_template/meshes/upperarm.STL
- added link right/upperarm_biceps_pulley, mass 0.01522; collision mesh filename=package://gummi_rightbase_template/meshes/upperarm_biceps_p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; visual mesh filename=package://gummi_rightbase_template/meshes/upperarm_biceps_p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
- added link right/upperarm_preroll, mass 0.11889; collision mesh filename=package://gummi_rightbase_template/meshes/upperarm_preroll.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; visual mesh filename=package://gummi_rightbase_template/meshes/upperarm_preroll.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
- added link right/upperarm_triceps_pulley, mass 0.01522; collision mesh filename=package://gummi_rightbase_template/meshes/upperarm_triceps_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; visual mesh filename=package://gummi_rightbase_template/meshes/upperarm_triceps_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
- added link right/wrist, mass 0.0644774651698934; collision mesh filename=package://gummi_rightee_handshake/meshes/wrist.STL; visual mesh filename=package://gummi_rightee_handshake/meshes/wrist.STL
Joints:
- removed joint elbow
- removed joint fastswitch
- removed joint forearm_roll
- removed joint gripper
- removed joint i1f
- removed joint i2f
- removed joint i3f
- removed joint i4f
- removed joint i5f
- removed joint shoulder_pitch
- removed joint shoulder_pitch_back_pulley_joint
- removed joint shoulder_pitch_pulley_front_joint
- removed joint shoulder_roll
- removed joint shoulder_roll_bottom_pulley
- removed joint shoulder_roll_top_pulley_joint
- removed joint shoulder_yaw
- removed joint upperarm_biceps_pulley_joint
- removed joint upperarm_roll
- removed joint upperarm_triceps_pulley_joint
- removed joint wrist_pitch
- added joint right/elbow: type revolute, parent right/upperarm, child right/lowerarm_preroll_u, origin xyz=-0.006 0.0184 -0.23533 rpy=0 0 0, axis 0 -1 0, limit lower=-0.75 upper=0.35 effort=0 velocity=0
- added joint right/fastswitch: type fixed, parent right/lowerarm_preroll_u, child right/lowerarm_preroll_d, origin xyz=0.056236 -0.019 -0.006 rpy=0 0 0, axis 0 0 0
- added joint right/forearm_roll: type continuous, parent right/lowerarm_preroll_d, child right/lowerarm, origin xyz=0.043506 -0.00023376 -0.019876 rpy=0 0 0, axis -1 0 0, limit effort=0 velocity=1
- added joint right/gripper: type revolute, parent right/wrist, child right/dummygripper, origin xyz=0 0 0 rpy=0 0 0, axis 0 1 0, limit lower=0 upper=2 effort=0 velocity=0
- added joint right/i1f: type revolute, parent right/wrist, child right/i1, origin xyz=0.059922 -0.031986 0.0029515 rpy=-0.79367 0.12795 -0.91441, axis 0 -1 0, limit lower=0 upper=0.8 effort=0 velocity=0, mimic joint=right/gripper
- added joint right/i2f: type revolute, parent right/wrist, child right/i2, origin xyz=0.12886 -0.0060786 -0.0024749 rpy=-6.9389E-16 -8.4436E-17 -0.12109, axis 0 -1 0, limit lower=0 upper=0.8 effort=0 velocity=0, mimic joint=right/gripper
- added joint right/i3f: type revolute, parent right/wrist, child right/i3, origin xyz=0.13223 0.0086295 -0.0025 rpy=-1.0408E-15 -5.7778E-30 -5.5511E-15, axis 0 -1 0, limit lower=0 upper=0.8 effort=0 velocity=0, mimic joint=right/gripper
- added joint right/i4f: type revolute, parent right/wrist, child right/i4, origin xyz=0.13046 0.023543 -0.0025 rpy=-1.0408E-15 1.4051E-16 0.13418, axis 0 -1 0, limit lower=0 upper=0.8 effort=0 velocity=0, mimic joint=right/gripper
- added joint right/i5f: type revolute, parent right/wrist, child right/i5, origin xyz=0.12703 0.037692 -0.0025 rpy=1.9429E-14 -3.8109E-15 0.19369, axis 0 -1 0, limit lower=0 upper=0.8 effort=0 velocity=0, mimic joint=right/gripper
- added joint right/shoulder_pitch: type revolute, parent right/shoulder, child right/upperarm_preroll, origin xyz=-0.024 -0.17679 8.6827E-05 rpy=0 0 0, axis -1 0 0, limit lower=-0.15 upper=1.1 effort=0 velocity=0
- added joint right/shoulder_pitch_back_pulley_joint: type fixed, parent right/shoulder_preroll, child right/shoulder_pitch_back_pulley, origin xyz=-0.067526 -0.024095 0.044 rpy=0 0 0, axis 0 0 0
- added joint right/shoulder_pitch_pulley_front_joint: type fixed, parent right/shoulder_preroll, child right/shoulder_pitch_front_pulley, origin xyz=0.067474 -0.024095 0.044 rpy=0 0 0, axis 0 0 0
- added joint right/shoulder_roll: type revolute, parent right/shoulder_preroll, child right/shoulder, origin xyz=-2.6378E-05 0.057605 0.1302 rpy=0 0 0, axis 0 -1 0, limit lower=-0.95 upper=2.3 effort=0 velocity=0
- added joint right/shoulder_roll_bottom_pulley: type fixed, parent right/shoulder, child right/shoulder_roll_bottom_pulley, origin xyz=-0.0208 -0.06848 -0.043 rpy=0 0 0, axis 0 0 -1, limit effort=0 velocity=0
- added joint right/shoulder_roll_top_pulley_joint: type fixed, parent right/shoulder, child right/shoulder_roll_top_pulley, origin xyz=0.0208 -0.06848 0.043 rpy=0 0 0, axis 0 0 0
- added joint right/shoulder_yaw: type revolute, parent right/base_link, child right/shoulder_preroll, origin xyz=-0.00027025 -0.10997 0.008 rpy=0 0 0, axis 0 0 1, limit lower=-0.75 upper=1 effort=0 velocity=0
- added joint right/upperarm_biceps_pulley_joint: type fixed, parent right/upperarm, child right/upperarm_biceps_pulley, origin xyz=0.0375 0 -0.10243 rpy=0 0 0, axis 0 0 0
- added joint right/upperarm_roll: type revolute, parent right/upperarm_preroll, child right/upperarm, origin xyz=0.056992 -0.010088 -0.035587 rpy=0 0 0, axis 0 0 -1, limit lower=-1.56 upper=1.56 effort=0 velocity=0
- added joint right/upperarm_triceps_pulley_joint: type fixed, parent right/upperarm, child right/upperarm_triceps_pulley, origin xyz=-0.0435 0 -0.12843 rpy=0 0 0, axis -1 0 0, limit effort=0 velocity=0
- added joint right/wrist_pitch: type revolute, parent right/lowerarm, child right/wrist, origin xyz=0.1511 -0.01935 0.0048471 rpy=0 0 0, axis 0 1 0, limit lower=-1 upper=1 effort=0 velocity=0
- joint leftbase_displacement: origin xyz=-0.2 0 0 rpy=-3.14 0 0 -> xyz=-0.2 0 0 rpy=0 0 0
- joint rightbase_displacement: child right_base_link -> right/base_link; origin xyz=0.2 0 0 rpy=0 0 0 -> xyz=0.2 0 0 rpy=-3.14 0 0

File: xacro/gummi_rig.urdf.xacro (robot description, xacro)
@@ -6,11 +6,11 @@
 <link name="base_link"/>
 <joint name="rightbase_displacement" type="fixed">
-  <origin rpy="0 0 0" xyz="0.2 0 0"/>
+  <origin rpy="-3.14 0 0" xyz="0.2 0 0"/>
   <parent link="base_link"/>
-  <child link="right_base_link"/>
+  <child link="right/base_link"/>
   <axis xyz="0 0 0"/>
 </joint>
 <joint name="leftbase_displacement" type="fixed">
-  <origin rpy="-3.14 0 0" xyz="-0.2 0 0"/>
+  <origin rpy="0 0 0" xyz="-0.2 0 0"/>
   <parent link="base_link"/>
   <child link="left/base_link"/>
